File: Hardware/LinuxCore/LinuxCore.kicad_pcb (KiCad board)
At the start: 2 copper layers, 52.5 x 57.4 mm, 153 parts, among them J1 USB_B_Micro, J2 USB_B_Micro, J3 Conn_02x15_Odd_Even, Q1 MMBT3904, Q2 MMBT3904, SW1 SW_Push, SW2 SW_Push, U1 NUC980DK61YC, U2 RLT8188_WIFI_MODUL, U3 TPS562200, U4 TPS562200, U5 TPS562200, U6 CP2102N-Axx-xQFN28, U7 W25Q128JVS, U8 L-KLS1-TF-003, Y1 Crystal, Y2 Crystal_GND24

Commit message: Update Board
Other:
- board text added: "+"
- board text added: "-"
- board text added: "PG8"
- board text added: "PG9"
- board text added: "PG9/PG8/If Botting From QSPI (-)/(-)/SPI-NAND, 1-bit (-)/(+)/SPI-NAND, 4-bit (+)/(-)/SPI-NOR, 4-bit (+)/(+)/SPI-NOR, 1-bit"
- board text added: "RESET"
- board text added: "SD0-BOOT"
