File: Hardware/LinuxCore/user.kicad_sch (KiCad schematic)
At the start: 7 parts, among them J3 Conn_02x15_Odd_Even

Commit message: update
Other:
- note added: "I2C 3 SCL"
- note added: "I2C 3 SDA"
- note added: "LCD-DC"
- note added: "PEN_IRQ_PIN"
- note added: "PWM1 CH 0"
- note added: "PWM1 CH 1"
- note added: "SPI0-CLK"
- note added: "SPI0-MISO"
- note added: "SPI0-MOSI"
- note added: "SPI0-SS"
- note added: "SPI0-SS1"
- note added: "UART 1 RX"
- note added: "UART 1 TX"
