File: Hardware/LinuxCore-v2/LinuxCore-v2.kicad_sch (KiCad schematic)
At the start: 0 parts

Commit message: update 3d model
Other:
- note added: "@0x6C heartbeat trigger"
- note added: "@0x6D cpu trigger"
- note added: "@0xA8 activity trigger"
- note added: "@0xA9 default on trigger"
Changed lines of the file:
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@@
+		)
+	)
+	(text "@0x6D cpu trigger"
+		(exclude_from_sim no)
+		(at 256.032 119.126 0)
+		(effects
+			(font
+				(size 1.27 1.27)
+			)
 		)
 	)
@@
 		)
 	)
+	(text "@0x6C heartbeat trigger"
+		(exclude_from_sim no)
+		(at 258.572 116.84 0)
+		(effects
+			(font
+				(size 1.27 1.27)
+			)
+		)
+	)
 	(text "@VCAP1_DATA3"
 		(exclude_from_sim no)
@@
 		)
 	)
+	(text "@0xA9 default on trigger"
+		(exclude_from_sim no)
+		(at 259.334 123.19 0)
+		(effects
+			(font
+				(size 1.27 1.27)
+			)
+		)
+	)
 	(text "@DATA7\n"
 		(exclude_from_sim no)
@@
 		)
 	)
+	(text "@0xA8 activity trigger"
+		(exclude_from_sim no)
+		(at 257.81 121.158 0)
+		(effects
+			(font
+				(size 1.27 1.27)
+			)
+		)
+	)
