File: Hardware/LinuxCore-v2/nau8822.kicad_sch (KiCad schematic)
At the start: 27 parts, among them U6 NAU88C22

Commit message: update 3d model
Parts:
- C44: value 10uF -> 33pF
- R43, R44: value 33R -> 10K
Changed lines of the file:
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@@
 		(fields_autoplaced yes)
 		(property "Reference" "R43"
-			(at 43.815 160.655 0)
+			(at 43.18 160.0199 0)
 			(effects
 				(font
@@
 			)
 		)
-		(property "Value" "33R"
-			(at 43.815 163.195 0)
+		(property "Value" "10K"
+			(at 43.18 162.5599 0)
 			(effects
 				(font
@@
 		(fields_autoplaced yes)
 		(property "Reference" "C44"
-			(at 83.185 160.655 0)
+			(at 82.55 160.0199 0)
 			(effects
 				(font
@@
 			)
 		)
-		(property "Value" "10uF"
-			(at 83.185 163.195 0)
+		(property "Value" "33pF"
+			(at 82.55 162.5599 0)
 			(effects
 				(font
@@
 		(fields_autoplaced yes)
 		(property "Reference" "R44"
-			(at 52.705 160.655 0)
+			(at 52.07 160.0199 0)
 			(effects
 				(font
@@
 			)
 		)
-		(property "Value" "33R"
-			(at 52.705 163.195 0)
+		(property "Value" "10K"
+			(at 52.07 162.5599 0)
 			(effects
 				(font
@@
 		(fields_autoplaced yes)
 		(property "Reference" "C44"
-			(at 71.755 160.655 0)
+			(at 71.12 160.0199 0)
 			(effects
 				(font
@@
 			)
 		)
-		(property "Value" "10uF"
-			(at 71.755 163.195 0)
-			(effects
-				(font
+		(property "Value" "33pF"
+			(at 71.12 162.5599 0)
+			(effects
+				(font
