File: Hardware/LinuxCore-v2/peripherals.kicad_sch (KiCad schematic)
At the start: 8 parts

Commit message: update 3d model
Parts:
- D3: value LED -> RED
- D4, D5: value LED -> BLUE
- D6: value LED -> GREEN
- R60: value 1K -> 2K
Changed lines of the file:
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@@
 			)
 		)
-		(property "Value" "LED"
+		(property "Value" "BLUE"
 			(at 53.6575 68.58 0)
 			(effects
@@
 			)
 		)
-		(property "Value" "1K"
+		(property "Value" "2K"
 			(at 67.31 48.26 90)
 			(effects
@@
 		(fields_autoplaced yes)
 		(property "Reference" "D6"
-			(at 54.2925 45.085 0)
-			(effects
-				(font
-					(size 1.27 1.27)
-				)
-			)
-		)
-		(property "Value" "LED"
-			(at 54.2925 47.625 0)
+			(at 54.2925 44.45 0)
+			(effects
+				(font
+					(size 1.27 1.27)
+				)
+			)
+		)
+		(property "Value" "GREEN"
+			(at 54.2925 46.99 0)
 			(effects
 				(font
@@
 			)
 		)
-		(property "Value" "LED"
+		(property "Value" "RED"
 			(at 53.6575 58.42 0)
 			(effects
@@
 			)
 		)
-		(property "Value" "LED"
+		(property "Value" "BLUE"
 			(at 54.2925 36.83 0)
 			(effects
