File: Hardware/LinuxCore-v2/usb_host_device.kicad_sch (KiCad schematic)
At the start: 5 parts, among them J6 USB_A_Stacked

Commit message: update 3d model
Parts:
- R56, R57, R58, R59: value 5.1K -> 33R
Changed lines of the file:
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@@
 			)
 		)
-		(property "Value" "5.1K"
+		(property "Value" "33R"
 			(at 154.305 90.17 90)
 			(effects
@@
 			)
 		)
-		(property "Value" "5.1K"
+		(property "Value" "33R"
 			(at 154.305 80.01 90)
 			(effects
@@
 			)
 		)
-		(property "Value" "5.1K"
+		(property "Value" "33R"
 			(at 154.305 95.25 90)
 			(effects
@@
 			)
 		)
-		(property "Value" "5.1K"
+		(property "Value" "33R"
 			(at 154.305 85.09 90)
 			(effects
